File: hardware/schematic/KiCad/rescue-backup/NewMain-2019-05-08-13-40-19.sch (KiCad schematic (older format))
At the start: 16 parts, among them J1 MDB, J2-1 Conn_01x01, J2-2 Conn_01x01, J2-3 Conn_01x01, J2-4 Conn_01x01, Q1 BC807, Q2 BC807, Q3 2N7002, U1 DC24V-DC5V

Commit message: update
Parts:
- removed U1: DC24V-DC5V, symbol custom-modules:DC24V-DC5V
- added psu?: dc24-dc5-module, symbol Converter_DCDC:dc24-dc5-module
Changed lines of the file:
@@
 EESchema Schematic File Version 4
-LIBS:NewMain-cache
 EELAYER 29 0
 EELAYER END
@@
 L power:GND #PWR013
 U 1 1 5B09563E
-P 2350 5000
-F 0 "#PWR013" H 2350 4750 50  0001 C CNN
-F 1 "GND" H 2350 4850 50  0000 C CNN
-F 2 "" H 2350 5000 50  0001 C CNN
-F 3 "" H 2350 5000 50  0001 C CNN
-	1    2350 5000
+P 2350 4950
+F 0 "#PWR013" H 2350 4700 50  0001 C CNN
+F 1 "GND" H 2350 4800 50  0000 C CNN
+F 2 "" H 2350 4950 50  0001 C CNN
+F 3 "" H 2350 4950 50  0001 C CNN
+	1    2350 4950
 	1    0    0    -1
 $EndComp
@@
 L power:GND #PWR014
 U 1 1 5B095685
-P 3500 5000
-F 0 "#PWR014" H 3500 4750 50  0001 C CNN
-F 1 "GND" H 3500 4850 50  0000 C CNN
-F 2 "" H 3500 5000 50  0001 C CNN
-F 3 "" H 3500 5000 50  0001 C CNN
-	1    3500 5000
+P 3350 4950
+F 0 "#PWR014" H 3350 4700 50  0001 C CNN
+F 1 "GND" H 3350 4800 50  0000 C CNN
+F 2 "" H 3350 4950 50  0001 C CNN
+F 3 "" H 3350 4950 50  0001 C CNN
+	1    3350 4950
 	1    0    0    -1
 $EndComp
@@
 L power:+5V #PWR015
 U 1 1 5B095758
-P 3500 4700
-F 0 "#PWR015" H 3500 4550 50  0001 C CNN
-F 1 "+5V" H 3500 4840 50  0000 C CNN
-F 2 "" H 3500 4700 50  0001 C CNN
-F 3 "" H 3500 4700 50  0001 C CNN
-	1    3500 4700
+P 3350 4550
+F 0 "#PWR015" H 3350 4400 50  0001 C CNN
+F 1 "+5V" H 3350 4690 50  0000 C CNN
+F 2 "" H 3350 4550 50  0001 C CNN
+F 3 "" H 3350 4550 50  0001 C CNN
+	1    3350 4550
 	1    0    0    -1
 $EndComp
@@
 L power:+24V #PWR016
 U 1 1 5B0957B3
-P 2350 4700
-F 0 "#PWR016" H 2350 4550 50  0001 C CNN
-F 1 "+24V" H 2350 4840 50  0000 C CNN
-F 2 "" H 2350 4700 50  0001 C CNN
-F 3 "" H 2350 4700 50  0001 C CNN
-	1    2350 4700
+P 2350 4550
+F 0 "#PWR016" H 2350 4400 50  0001 C CNN
+F 1 "+24V" H 2350 4690 50  0000 C CNN
+F 2 "" H 2350 4550 50  0001 C CNN
+F 3 "" H 2350 4550 50  0001 C CNN
+	1    2350 4550
 	1    0    0    -1
 $EndComp
@@
 	6600 1800 6550 1800
 $Comp
-L power:+3.3V #PWR0101
+L power:+3.3V #PWR?
 U 1 1 5B2CA167
 P 6600 1800
-F 0 "#PWR0101" H 6600 1650 50  0001 C CNN
+F 0 "#PWR?" H 6600 1650 50  0001 C CNN
 F 1 "+3.3V" H 6600 1940 50  0000 C CNN
 F 2 "" H 6600 1800 50  0001 C CNN
@@
 $EndComp
 $Comp
-L power:GND #PWR0102
+L power:GND #PWR?
 U 1 1 5B2CAFCD
 P 7150 4400
-F 0 "#PWR0102" H 7150 4150 50  0001 C CNN
+F 0 "#PWR?" H 7150 4150 50  0001 C CNN
 F 1 "GND" H 7150 4250 50  0000 C CNN
 F 2 "" H 7150 4400 50  0001 C CNN
@@
 	7150 3900 7100 3900
 $Comp
-L custom-modules:DC24V-DC5V U1
-U 1 1 5CD2F1A2
-P 2950 4850
-F 0 "U1" H 2925 5287 60  0000 C CNN
-F 1 "DC24V-DC5V" H 2925 5181 60  0000 C CNN
-F 2 "" H 2850 4550 60  0001 C CNN
-F 3 "" H 2850 4550 60  0001 C CNN
-	1    2950 4850
-	1    0    0    -1
-$EndComp
+L Converter_DCDC:dc24-dc5-module psu?
+U 1 1 5CD320C8
+P 2850 4750
+F 0 "psu?" H 2850 5217 50  0000 C CNN
+F 1 "dc24-dc5-module" H 2850 5126 50  0000 C CNN
+F 2 "" H 2850 5150 50  0001 C CNN
+F 3 "" H 2850 5150 50  0001 C CNN
+	1    2850 4750
+	1    0    0    -1
+$EndComp
