File: hardware/evend-adapter/kicad/evend-adapter/evend-adapter.kicad_pcb (KiCad board)
At the start: 2 copper layers, 122.4 x 69.1 mm, 41 parts, among them J1 Orange_pi_lite, J2 Keyboard, J3 Conn_02x03_Top_Bottom, Q2 BC807, Q3 BC807, Q4 2N7002, Q5 2N7002, Q6 2N7002, U1 RC1602A, X1 Arduino_Pro_Mini-1

Commit message: pcb release v1.0
Parts:
- added R25: 300, evend-adapter:C_1206_1-HandSoldering, B.Cu at (128.0, 165.8)
- added R26: 1.5k, evend-adapter:C_1206_1-HandSoldering, B.Cu at (134.6, 161.8)
- o1, o2, o3, o4, o5, o6, o7: footprint evend-adapter:L_1806_Handsoldering -> evend-adapter:C_1206_HandSoldering
- moved J2 62.6 mm to (96.8, 169.7)
- moved R8 4.20 mm to (83.1, 144.3)
- moved Q6 2.24 mm to (101.1, 158.8)
- moved R9 2.21 mm to (83.1, 146.1)
- moved R24 1.59 mm to (98.1, 157.0), turned to 180 degrees
- moved o3 0.51 mm to (99.1, 153.2)
- moved o4 0.38 mm to (104.6, 144.4)
- moved R5 0.35 mm to (79.1, 144.3)
- moved o2 0.21 mm to (94.8, 149.4)
- moved o5 0.17 mm to (84.4, 154.9)
- renumbered +6V to J4, GND to J5
Connections:
- J1 pad 2: +5V -> (no net)
- J2 pad 1: SDA -> SCL
- J2 pad 2: SCL -> SDA
- J2 pad 4: +5V -> +5VD
- R8 pad 2: SDA -> SCL
- R9 pad 2: SCL -> SDA
- U1 pad 2: +5V -> +5VD
Routing:
- net GND: track 309.1 -> 213.7 mm
- net SCL: track 111.5 -> 41.0 mm
- net +5V: track 68.0 -> 0.00 mm
- net +6V: track 108.3 -> 171.1 mm
- net SDA: track 101.2 -> 51.5 mm
- net +5VD: track 0.00 -> 45.2 mm
- net SS-5V: track 22.8 -> 13.5 mm
- net Net-(Q6-Pad1): track 5.73 -> 1.81 mm
- net MDB-MT: track 58.5 -> 60.8 mm
- net SS-3V: track 91.9 -> 93.7 mm
- net MOSI-5V: track 5.93 -> 7.66 mm
- net Net-(Q2-Pad3): track 15.8 -> 17.5 mm
- net D6: track 49.9 -> 51.4 mm
- net D5: track 45.3 -> 46.8 mm
- net D4: track 41.7 -> 43.2 mm
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