File: hardware/evend-adapter/kicad/evend-adapter/evend-adapter.kicad_pcb (KiCad board)
At the start: 2 copper layers, 122.4 x 69.1 mm, 43 parts, among them J1 Orange_pi_lite, J2 Keyboard, J3 Conn_02x03_Top_Bottom, J4 Conn_01x01_Female, J5 Conn_01x01_Female, Q2 BC807, Q3 BC807, Q4 2N7002, Q5 2N7002, Q6 2N7002, U1 RC1602A, X1 Arduino_Pro_Mini-1

Commit message: -
Parts:
- removed D1: B260, Diodes_SMD:D_1206
- removed R25: 300, evend-adapter:C_1206_1-HandSoldering
- removed R26: 1.5k, evend-adapter:C_1206_1-HandSoldering
- R6: value 10K -> 10k; moved to F.Cu
- moved R6 0.22 mm to (78.2, 141.2)
Connections:
- J2 pad 4: +5VD -> +5V
- J3 pad 1: Net-(D1-Pad2) -> MDB+24V
- J4 pad 1: +6V -> +5V
- Q2 pad 2: +5C -> +5V
- R13 pad 1: +5C -> +5V
- R15 pad 1: +5C -> +5V
- R23 pad 1: +5C -> +5V
- R24 pad 1: +5C -> +5V
- R3 pad 1: +5C -> +5V
- R5 pad 1: +5C -> +5V
- R8 pad 1: +5C -> +5V
- R9 pad 1: +5C -> +5V
- U1 pad 2: +5VD -> +5V
- X1 pad 1A: +6V -> (no net)
- X1 pad 4A: +5C -> +5V
- o2 pad 2: +5C -> +5V
- psu1 pad 4: +6V -> +5V
Routing:
- net +5V: track 0.00 -> 90.8 mm
- net Net-(D1-Pad2): track 50.2 -> 0.00 mm
- net MDB+24V: track 21.0 -> 71.2 mm
- net +5C: track 55.4 -> 9.77 mm
- net +5VD: track 45.2 -> 0.00 mm
- net Net-(Q6-Pad1): track 1.81 -> 3.50 mm
