File: hardware/schematic/evend-adapter/kicad/evend-adapter/evend-adapter.sch (KiCad schematic (older format))
At the start: 40 parts, among them J1 Orange_pi_lite, J2 Keyboard, J3 Conn_02x03_Top_Bottom, J4 Conn_01x01_Female, J5 Conn_01x01_Female, Q2 BC807, Q3 BC807, Q4 2N7002, Q5 2N7002, Q6 2N7002, U1 RC1602A, X1 Arduino_Pro_Mini-1

Commit message: update hardware data
Parts:
- added U?: CR2013-MI2120, Display:CR2013-MI2120, symbol Driver_Display:CR2013-MI2120
Connections:
- net +5V: now also U?.1 (VCC)
- net GND: now also U?.2 (GND)
- net MOSI-3V: now also U?.6 (MOSI)
- net SCK-3V: now also U?.7 (SCK)
- net TFT-LED: now reaches J1.31 (8)
- net TFT-LED: now also U?.8 (LED)
- net TFT-DС: now reaches J1.33 (9)
- net TFT-DС: now also U?.5 (D/~C)
- net TFT-RESET: now reaches J1.35 (10)
- net TFT-RESET: now also U?.4 (RESET)
- net TFT-CS: now reaches J1.37 (20)
- net TFT-CS: now also U?.3 (~CS)
- no-connect marks 33 -> 35
Changed lines of the file:
@@
 NoConn ~ 3600 5450
 NoConn ~ 5850 5750
-NoConn ~ 3600 5550
-NoConn ~ 3600 5750
-NoConn ~ 3600 5650
 NoConn ~ 5850 5950
 NoConn ~ 5850 4750
-NoConn ~ 3600 5950
+NoConn ~ 3600 5550
 NoConn ~ 5850 5050
 NoConn ~ 5850 5850
@@
 NoConn ~ 5850 4250
 NoConn ~ 5850 5550
-NoConn ~ 3600 5850
 $Comp
 L Device:R R5
@@
 	0    -1   -1   0
 $EndComp
-Wire Wire Line
-	6550 950  6950 950
 Connection ~ 7300 950
 Wire Wire Line
@@
 L power:+5C #PWR0120
 U 1 1 5D07A396
-P 7700 950
-F 0 "#PWR0120" H 7700 800 50  0001 C CNN
-F 1 "+5C" H 7715 1078 50  0000 L CNN
-F 2 "" H 7700 950 50  0001 C CNN
-F 3 "" H 7700 950 50  0001 C CNN
-	1    7700 950
+P 7700 850
+F 0 "#PWR0120" H 7700 700 50  0001 C CNN
+F 1 "+5C" H 7715 978 50  0000 L CNN
+F 2 "" H 7700 850 50  0001 C CNN
+F 3 "" H 7700 850 50  0001 C CNN
+	1    7700 850
 	1    0    0    -1
 $EndComp
@@
 	1    0    0    -1
 $EndComp
-Connection ~ 6950 950
 $Comp
 L power:GND #PWR0134
@@
 $EndComp
 $Comp
-L power:+5V #PWR?
+L power:+5V #PWR0102
 U 1 1 5DA08F9F
 P 5200 1050
-F 0 "#PWR?" H 5200 900 50  0001 C CNN
+F 0 "#PWR0102" H 5200 900 50  0001 C CNN
 F 1 "+5V" V 5200 1250 50  0000 C CNN
 F 2 "" H 5200 1050 50  0001 C CNN
@@
 $EndComp
 $Comp
-L power:+5V #PWR?
+L power:+5V #PWR0106
 U 1 1 5DA0A4F8
 P 3850 2700
-F 0 "#PWR?" H 3850 2550 50  0001 C CNN
+F 0 "#PWR0106" H 3850 2550 50  0001 C CNN
 F 1 "+5V" H 3850 2900 50  0000 C CNN
 F 2 "" H 3850 2700 50  0001 C CNN
@@
 $EndComp
 $Comp
-L power:+5V #PWR?
+L power:+5V #PWR0109
 U 1 1 5DA12A11
 P 7700 1900
-F 0 "#PWR?" H 7700 1750 50  0001 C CNN
+F 0 "#PWR0109" H 7700 1750 50  0001 C CNN
 F 1 "+5V" H 7700 2100 50  0000 C CNN
 F 2 "" H 7700 1900 50  0001 C CNN
@@
 $EndComp
 $Comp
-L power:+5V #PWR?
+L power:+5V #PWR0111
 U 1 1 5DA12C50
 P 8050 750
-F 0 "#PWR?" H 8050 600 50  0001 C CNN
+F 0 "#PWR0111" H 8050 600 50  0001 C CNN
 F 1 "+5V" H 8050 950 50  0000 C CNN
 F 2 "" H 8050 750 50  0001 C CNN
@@
 $EndComp
 $Comp
-L power:+5V #PWR?
+L power:+5V #PWR0112
 U 1 1 5DA1314C
 P 10000 800
-F 0 "#PWR?" H 10000 650 50  0001 C CNN
+F 0 "#PWR0112" H 10000 650 50  0001 C CNN
 F 1 "+5V" H 10000 1000 50  0000 C CNN
 F 2 "" H 10000 800 50  0001 C CNN
@@
 $EndComp
 $Comp
-L power:+5V #PWR?
+L power:+5V #PWR0113
 U 1 1 5DA13677
 P 9650 2400
-F 0 "#PWR?" H 9650 2250 50  0001 C CNN
+F 0 "#PWR0113" H 9650 2250 50  0001 C CNN
 F 1 "+5V" H 9650 2600 50  0000 C CNN
 F 2 "" H 9650 2400 50  0001 C CNN
@@
 $EndComp
 $Comp
-L power:+5V #PWR?
+L power:+5V #PWR0115
 U 1 1 5DA13B3F
 P 7700 2750
-F 0 "#PWR?" H 7700 2600 50  0001 C CNN
+F 0 "#PWR0115" H 7700 2600 50  0001 C CNN
 F 1 "+5V" H 7700 2950 50  0000 C CNN
 F 2 "" H 7700 2750 50  0001 C CNN
@@
 	3850 2750 3850 3000
 $Comp
-L power:+5V #PWR?
+L power:+5V #PWR0117
 U 1 1 5DA1A493
-P 2550 3050
-F 0 "#PWR?" H 2550 2900 50  0001 C CNN
-F 1 "+5V" V 2550 3250 50  0000 C CNN
-F 2 "" H 2550 3050 50  0001 C CNN
-F 3 "" H 2550 3050 50  0001 C CNN
-	1    2550 3050
-	0    1    1    0
-$EndComp
-$Comp
-L power:+5V #PWR?
+P 2750 3050
+F 0 "#PWR0117" H 2750 2900 50  0001 C CNN
+F 1 "+5V" V 2750 3250 50  0000 C CNN
+F 2 "" H 2750 3050 50  0001 C CNN
+F 3 "" H 2750 3050 50  0001 C CNN
+	1    2750 3050
+	0    1    1    0
+$EndComp
+$Comp
+L power:+5V #PWR0119
 U 1 1 5DA1A9F5
 P 1950 5500
-F 0 "#PWR?" H 1950 5350 50  0001 C CNN
+F 0 "#PWR0119" H 1950 5350 50  0001 C CNN
 F 1 "+5V" H 1950 5700 50  0000 C CNN
 F 2 "" H 1950 5500 50  0001 C CNN
@@
 	1250 900  1550 900
 $Comp
-L power:+5V #PWR?
+L power:+5V #PWR0121
 U 1 1 5DA2030B
 P 5200 1950
-F 0 "#PWR?" H 5200 1800 50  0001 C CNN
+F 0 "#PWR0121" H 5200 1800 50  0001 C CNN
 F 1 "+5V" V 5200 2150 50  0000 C CNN
 F 2 "" H 5200 1950 50  0001 C CNN
@@
 $EndComp
 NoConn ~ 5850 4150
+Wire Wire Line
+	7700 850  7700 950
+Wire Wire Line
+	2350 3050 2550 3050
+Connection ~ 2550 3050
+Wire Wire Line
+	2550 3050 2750 3050
+Text GLabel 5500 7000 2    60   Input ~ 0
+MOSI-3V
+$Comp
+L Driver_Display:CR2013-MI2120 U?
+U 1 1 5E2A8BE3
+P 4700 7000
+F 0 "U?" H 4900 7600 50  0000 C CNN
+F 1 "CR2013-MI2120" H 4350 7600 50  0000 C CNN
+F 2 "Display:CR2013-MI2120" H 4700 6300 50  0001 C CNN
+F 3 "http://pan.baidu.com/s/11Y990" H 4050 7500 50  0001 C CNN
+	1    4700 7000
+	1    0    0    -1
+$EndComp
+Text GLabel 5500 7300 2    60   Input ~ 0
+TFT-CS
+Text GLabel 5500 7200 2    60   Input ~ 0
+TFT-RESET
+Text GLabel 5500 7100 2    60   Input ~ 0
+TFT-DС
+Text GLabel 5500 6800 2    60   Input ~ 0
+TFT-LED
+Text GLabel 5500 6900 2    60   Input ~ 0
+SCK-3V
+Text GLabel 3600 5950 0    60   Input ~ 0
+TFT-CS
+Text GLabel 3600 5850 0    60   Input ~ 0
+TFT-RESET
+Text GLabel 3600 5750 0    60   Input ~ 0
+TFT-DС
+Text GLabel 3600 5650 0    60   Input ~ 0
+TFT-LED
+NoConn ~ 3900 6600
+NoConn ~ 3900 6700
+NoConn ~ 3900 6800
+NoConn ~ 3900 6900
+NoConn ~ 3900 7000
+NoConn ~ 5500 6700
+$Comp
+L power:+5V #PWR?
+U 1 1 5E2BFA20
+P 4700 6400
+F 0 "#PWR?" H 4700 6250 50  0001 C CNN
+F 1 "+5V" H 4700 6600 50  0000 C CNN
+F 2 "" H 4700 6400 50  0001 C CNN
+F 3 "" H 4700 6400 50  0001 C CNN
+	1    4700 6400
+	1    0    0    -1
+$EndComp
+$Comp
+L power:GND #PWR?
+U 1 1 5E2C0269
+P 4700 7600
+F 0 "#PWR?" H 4700 7350 50  0001 C CNN
+F 1 "GND" H 4700 7450 50  0000 C CNN
+F 2 "" H 4700 7600 50  0001 C CNN
+F 3 "" H 4700 7600 50  0001 C CNN
+	1    4700 7600
+	1    0    0    -1
+$EndComp
 $EndSCHEMATC
